File: pi4_pmod.kicad_sch (KiCad schematic)
At the start: 16 parts, among them J1 Pi-4 IO Extension, J2 5V, J3 uart, J4 pmod 1, J5 pmod 2, J6 camera

Commit message: add screenshots
Other:
- company: (none) -> S59MZ
- title: (none) -> Pi-4 PMOD Adapter
